Commit message: adding launch files for ros2 control

File: pick_and_place_description/urdf/turtlebot_arm.xacro (robot description, xacro)
@@ -1,5 +1,8 @@
 <?xml version="1.0"?>
-<robot name="robot_arm">
-  <link name="base_link"/>
+<robot name="robot_arm" xmlns:xacro="http://wiki.ros.org/xacro">
+  <xacro:arg name="use_gazebo" default="false" />
+  <xacro:arg name="use_ignition" default="false" />
+  <xacro:arg name="use_fake_hardware" default="false" />
+  <link name="base_link" />
   <link name="arm_base">
     <inertial>
@@ -38,6 +41,6 @@
       </geometry>
     </collision>
-</link>
-<link name="bicep">
+  </link>
+  <link name="bicep">
     <inertial>
       <origin
@@ -113,5 +116,5 @@
     </collision>
   </link>
- <link name="elbow">
+  <link name="elbow">
     <inertial>
       <origin
@@ -150,5 +153,5 @@
     </collision>
   </link>
-<link name="top_wrist">
+  <link name="top_wrist">
     <inertial>
       <origin
@@ -187,72 +190,89 @@
     </collision>
   </link>
-<!--######################################################################-->
-<joint name="arm_base_joint" type="continuous">
-  <axis xyz="0 0 1"/>
-  <parent link="base_link"/>
-  <child link="arm_base"/>
-  <origin rpy="0 0 0" xyz="0.0 0.0 0.1"/>
-</joint>
-<joint name="shoulder_joint" type="continuous">
-  <axis xyz="0 1 0"/>
-  <parent link="arm_base"/>
-  <child link="bicep"/>
-  <origin rpy="0 0 1.5708" xyz="-0.05166 0.0 0.20271"/>
-</joint>
-<joint name="bottom_wrist_joint" type="continuous">
-  <axis xyz="0 1 0"/>
-  <parent link="bicep"/>
-  <child link="bottom_wrist"/>
-  <origin rpy="0 0 0" xyz="0.0 -0.05194 0.269"/>
-</joint>
-<joint name="elbow_joint" type="fixed">
-  <!-- <axis xyz="0 0 1"/> -->
-  <parent link="bottom_wrist"/>
-  <child link="elbow"/>
-  <origin rpy="0 0 0" xyz="0.0 0 0.13522"/>
-</joint>
-<joint name="top_wrist_joint" type="continuous">
-  <axis xyz="0 1 0"/>
-  <parent link="elbow"/>
-  <child link="top_wrist"/>
-  <origin rpy="0 0 0" xyz="0.0 0 0.20994"/>
-</joint>
-<!--######################################################################-->
-<ros2_control name="robot_arm" type="system">
-  <hardware>
-    <plugin>mock_components/GenericSystem</plugin>
-  </hardware>
-  <joint name="arm_base_joint">
-    <command_interface name="position">
-      <param name="min">-1</param>
-      <param name="max">1</param>
-    </command_interface>
-    <state_interface name="position"/>
-    <state_interface name="velocity"/>
-  </joint>
-  <joint name="shoulder_joint">
-    <command_interface name="position">
-      <param name="min">-1</param>
-      <param name="max">1</param>
-    </command_interface>
-    <state_interface name="position"/>
-    <state_interface name="velocity"/>
-  </joint>
-  <joint name="bottom_wrist_joint">
-    <command_interface name="position">
-      <param name="min">-1</param>
-      <param name="max">1</param>
-    </command_interface>
-    <state_interface name="position"/>
-    <state_interface name="velocity"/>
-  </joint>
-  <joint name="top_wrist_joint">
-    <command_interface name="position">
-      <param name="min">-1</param>
-      <param name="max">1</param>
-    </command_interface>
-    <state_interface name="position"/>
-    <state_interface name="velocity"/>
-  </joint>
-</ros2_control>
+  <!--######################################################################-->
+  <joint name="arm_base_joint" type="continuous">
+    <axis xyz="0 0 1" />
+    <parent link="base_link" />
+    <child link="arm_base" />
+    <origin rpy="0 0 0" xyz="0.0 0.0 0.1" />
+  </joint>
+  <joint name="shoulder_joint" type="continuous">
+    <axis xyz="0 1 0" />
+    <parent link="arm_base" />
+    <child link="bicep" />
+    <origin rpy="0 0 1.5708" xyz="-0.05166 0.0 0.20271" />
+  </joint>
+  <joint name="bottom_wrist_joint" type="continuous">
+    <axis xyz="0 1 0" />
+    <parent link="bicep" />
+    <child link="bottom_wrist" />
+    <origin rpy="0 0 0" xyz="0.0 -0.05194 0.269" />
+  </joint>
+  <joint name="elbow_joint" type="fixed">
+    <!-- <axis xyz="0 0 1"/> -->
+    <parent link="bottom_wrist" />
+    <child link="elbow" />
+    <origin rpy="0 0 0" xyz="0.0 0 0.13522" />
+  </joint>
+  <joint name="top_wrist_joint" type="continuous">
+    <axis xyz="0 1 0" />
+    <parent link="elbow" />
+    <child link="top_wrist" />
+    <origin rpy="0 0 0" xyz="0.0 0 0.20994" />
+  </joint>
+  <!--######################################################################-->
+  <ros2_control name="robot_arm" type="system">
+    <hardware>
+      <xacro:if value="$(arg use_gazebo)">
+        <plugin>gazebo_ros2_control/GazeboSystem</plugin>
+      </xacro:if>
+      <xacro:if value="$(arg use_ignition)">
+        <plugin>ign_ros2_control/IgnitionSystem</plugin>
+      </xacro:if>
+      <xacro:if value="$(arg use_fake_hardware)">
+        <plugin>mock_components/GenericSystem</plugin>
+      </xacro:if>
+    </hardware>
+    <joint name="arm_base_joint">
+      <command_interface name="position">
+        <param name="min">-1</param>
+        <param name="max">1</param>
+      </command_interface>
+      <state_interface name="position" />
+      <state_interface name="velocity" />
+    </joint>
+    <joint name="shoulder_joint">
+      <command_interface name="position">
+        <param name="min">-1</param>
+        <param name="max">1</param>
+      </command_interface>
+      <state_interface name="position" />
+      <state_interface name="velocity" />
+    </joint>
+    <joint name="bottom_wrist_joint">
+      <command_interface name="position">
+        <param name="min">-1</param>
+        <param name="max">1</param>
+      </command_interface>
+      <state_interface name="position" />
+      <state_interface name="velocity" />
+    </joint>
+    <joint name="top_wrist_joint">
+      <command_interface name="position">
+        <param name="min">-1</param>
+        <param name="max">1</param>
+      </command_interface>
+      <state_interface name="position" />
+      <state_interface name="velocity" />
+    </joint>
+  </ros2_control>
+  <xacro:if value="$(arg use_gazebo)">
+    <gazebo reference="world">
+    </gazebo>
+    <gazebo>
+      <plugin filename="libgazebo_ros2_control.so" name="gazebo_ros2_control">
+        <parameters>$(find pick_and_place_description)/config/robot_controller.yaml</parameters>
+      </plugin>
+    </gazebo>
+  </xacro:if>
 </robot>

Commit message: Adding gazebo sim launch file

File: pick_and_place_description/urdf/turtlebot_arm.xacro (robot description, xacro)
@@ -4,5 +4,20 @@
   <xacro:arg name="use_ignition" default="false" />
   <xacro:arg name="use_fake_hardware" default="false" />
-  <link name="base_link" />
+  <link name="world" />
+  <link name="base_link">
+    <visual>
+      <geometry>
+        <box size="0.3 0.2 0.1"/>
+      </geometry>
+      <origin xyz="0 0 0"/>
+      <material name="green">
+        <color rgba="0 0.8 .8 1"/>
+      </material>
+    </visual>
+    <inertial>
+      <mass value="100"/>
+      <inertia ixx="1.0" ixy="0.0" ixz="0.0" iyy="1.0" iyz="0.0" izz="1.0"/>
+    </inertial>
+  </link>
   <link name="arm_base">
     <inertial>
@@ -25,5 +40,5 @@
         rpy="0 0 0" />
       <geometry>
-        <mesh filename="package://pick_and_place_description/meshes/arm_base.stl" />
+        <mesh filename="file://$(find pick_and_place_description)/meshes/arm_base.stl" />
       </geometry>
       <material
@@ -38,5 +53,5 @@
         rpy="0 0 0" />
       <geometry>
-        <mesh filename="package://pick_and_place_description/meshes/arm_base.stl" />
+        <mesh filename="file://$(find pick_and_place_description)/meshes/arm_base.stl" />
       </geometry>
     </collision>
@@ -62,5 +77,5 @@
         rpy="0 -1.5708 0" />
       <geometry>
-        <mesh filename="package://pick_and_place_description/meshes/bicep.stl" />
+        <mesh filename="file://$(find pick_and_place_description)/meshes/bicep.stl" />
       </geometry>
       <material
@@ -75,5 +90,5 @@
         rpy="0 -1.5708 0" />
       <geometry>
-        <mesh filename="package://pick_and_place_description/meshes/bicep.stl" />
+        <mesh filename="file://$(find pick_and_place_description)/meshes/bicep.stl" />
       </geometry>
     </collision>
@@ -99,5 +114,5 @@
         rpy="3.14 0 1.5708" />
       <geometry>
-        <mesh filename="package://pick_and_place_description/meshes/wrist.stl" />
+        <mesh filename="file://$(find pick_and_place_description)/meshes/wrist.stl" />
       </geometry>
       <material
@@ -112,5 +127,5 @@
         rpy="3.14 0 1.5708" />
       <geometry>
-        <mesh filename="package://pick_and_place_description/meshes/wrist.stl" />
+        <mesh filename="file://$(find pick_and_place_description)/meshes/wrist.stl" />
       </geometry>
     </collision>
@@ -136,5 +151,5 @@
         rpy="0 -1.5708 0" />
       <geometry>
-        <mesh filename="package://pick_and_place_description/meshes/elbow.stl" />
+        <mesh filename="file://$(find pick_and_place_description)/meshes/elbow.stl" />
       </geometry>
       <material
@@ -149,5 +164,5 @@
         rpy="0 -1.5708 0" />
       <geometry>
-        <mesh filename="package://pick_and_place_description/meshes/elbow.stl" />
+        <mesh filename="file://$(find pick_and_place_description)/meshes/elbow.stl" />
       </geometry>
     </collision>
@@ -173,5 +188,5 @@
         rpy="3.14 0 1.5708" />
       <geometry>
-        <mesh filename="package://pick_and_place_description/meshes/wrist.stl" />
+        <mesh filename="file://$(find pick_and_place_description)/meshes/wrist.stl" />
       </geometry>
       <material
@@ -186,14 +201,19 @@
         rpy="3.14 0 1.5708" />
       <geometry>
-        <mesh filename="package://pick_and_place_description/meshes/wrist.stl" />
+        <mesh filename="file://$(find pick_and_place_description)/meshes/wrist.stl" />
       </geometry>
     </collision>
   </link>
   <!--######################################################################-->
+  <joint name="base_joint" type="fixed">
+    <origin rpy="0 0 0" xyz="0 0 0" />
+    <parent link="world" />
+    <child link="base_link" />
+  </joint>
   <joint name="arm_base_joint" type="continuous">
     <axis xyz="0 0 1" />
     <parent link="base_link" />
     <child link="arm_base" />
-    <origin rpy="0 0 0" xyz="0.0 0.0 0.1" />
+    <origin rpy="0 0 0" xyz="0.0 0.0 0.0" />
   </joint>
   <joint name="shoulder_joint" type="continuous">
@@ -210,5 +230,5 @@
   </joint>
   <joint name="elbow_joint" type="fixed">
-    <!-- <axis xyz="0 0 1"/> -->
+    <axis xyz="0 0 1"/>
     <parent link="bottom_wrist" />
     <child link="elbow" />
@@ -239,6 +259,9 @@
         <param name="max">1</param>
       </command_interface>
-      <state_interface name="position" />
+      <state_interface name="position">
+        <param name="initial_value">0.0</param>
+      </state_interface>
       <state_interface name="velocity" />
+      <state_interface name="effort" />
     </joint>
     <joint name="shoulder_joint">
@@ -247,6 +270,9 @@
         <param name="max">1</param>
       </command_interface>
-      <state_interface name="position" />
+      <state_interface name="position">
+        <param name="initial_value">0.0</param>
+      </state_interface>
       <state_interface name="velocity" />
+      <state_interface name="effort" />
     </joint>
     <joint name="bottom_wrist_joint">
@@ -255,6 +281,9 @@
         <param name="max">1</param>
       </command_interface>
-      <state_interface name="position" />
+      <state_interface name="position">
+        <param name="initial_value">0.0</param>
+      </state_interface>
       <state_interface name="velocity" />
+      <state_interface name="effort" />
     </joint>
     <joint name="top_wrist_joint">
@@ -263,11 +292,12 @@
         <param name="max">1</param>
       </command_interface>
-      <state_interface name="position" />
+      <state_interface name="position">
+        <param name="initial_value">0.0</param>
+      </state_interface>
       <state_interface name="velocity" />
+      <state_interface name="effort" />
     </joint>
   </ros2_control>
   <xacro:if value="$(arg use_gazebo)">
-    <gazebo reference="world">
-    </gazebo>
     <gazebo>
       <plugin filename="libgazebo_ros2_control.so" name="gazebo_ros2_control">
@@ -276,3 +306,11 @@
     </gazebo>
   </xacro:if>
+  <xacro:if value="$(arg sim_ignition)">
+    <gazebo>
+      <plugin filename="libign_ros2_control-system.so" name="ign_ros2_control::IgnitionROS2ControlPlugin">
+        <parameters>$(find pick_and_place_description)/config/robot_controller.yaml</parameters>
+        <controller_manager_node_name>controller_manager</controller_manager_node_name>
+      </plugin>
+    </gazebo>
+  </xacro:if>
 </robot>
