Commit message: changed joint type

File: pick_and_place_description/urdf/robot_arm.xacro (robot description, xacro)
@@ -211,21 +211,24 @@
     <child link="base_link" />
   </joint>
-  <joint name="arm_base_joint" type="continuous">
+  <joint name="arm_base_joint" type="revolute">
     <axis xyz="0 0 1" />
     <parent link="base_link" />
     <child link="arm_base" />
     <origin rpy="0 0 0" xyz="0.0 0.0 0.0" />
-  </joint>
-  <joint name="shoulder_joint" type="continuous">
+    <limit effort="0" lower="-3.14" upper="3.14" velocity="3.67"/>
+  </joint>
+  <joint name="shoulder_joint" type="revolute">
     <axis xyz="0 1 0" />
     <parent link="arm_base" />
     <child link="bicep" />
     <origin rpy="0 0 1.5708" xyz="-0.05166 0.0 0.20271" />
-  </joint>
-  <joint name="bottom_wrist_joint" type="continuous">
+    <limit effort="0" lower="-3.14" upper="3.14" velocity="3.67"/>
+  </joint>
+  <joint name="bottom_wrist_joint" type="revolute">
     <axis xyz="0 1 0" />
     <parent link="bicep" />
     <child link="bottom_wrist" />
     <origin rpy="0 0 0" xyz="0.0 -0.05194 0.269" />
+    <limit effort="0" lower="-3.14" upper="3.14" velocity="3.67"/>
   </joint>
   <joint name="elbow_joint" type="fixed">
@@ -235,9 +238,10 @@
     <origin rpy="0 0 0" xyz="0.0 0 0.13522" />
   </joint>
-  <joint name="top_wrist_joint" type="continuous">
+  <joint name="top_wrist_joint" type="revolute">
     <axis xyz="0 1 0" />
     <parent link="elbow" />
     <child link="top_wrist" />
     <origin rpy="0 0 0" xyz="0.0 0 0.20994" />
+    <limit effort="0" lower="-3.14" upper="3.14" velocity="3.67"/>
   </joint>
   <!--######################################################################-->

Commit message: fixing gripper issues and adding depth camera

File: pick_and_place_description/urdf/robot_arm.xacro (robot description, xacro)
@@ -205,4 +205,19 @@
     </collision>
   </link>
+  <link name="camera_link">
+    <visual>
+      <geometry>
+        <box size="0.1 0.1 0.1"/>
+      </geometry>
+      <origin xyz="0 0 0"/>
+      <material name="green">
+        <color rgba="0 0.8 .8 1"/>
+      </material>
+    </visual>
+    <inertial>
+      <mass value="1"/>
+      <inertia ixx="1.0" ixy="0.0" ixz="0.0" iyy="1.0" iyz="0.0" izz="1.0"/>
+    </inertial>
+  </link>
   <!--######################################################################-->
   <joint name="base_joint" type="fixed">
@@ -244,4 +259,9 @@
     <origin rpy="0 0 0" xyz="0.0 0 0.20994" />
     <limit effort="0" lower="-3.14" upper="3.14" velocity="3.67"/>
+  </joint>
+  <joint name="camera_joint" type="fixed">
+    <origin rpy="0 1.57 0" xyz="0 0 1.2" />
+    <parent link="world" />
+    <child link="camera_link" />
   </joint>
   <!--######################################################################-->
@@ -310,6 +330,5 @@
       <plugin filename='libgazebo_ros_vacuum_gripper.so' name='vacuum_gripper'>
         <link_name>top_wrist</link_name>
-        <max_distance>5.0</max_distance>
-        <max_force>500</max_force>
+        <max_distance>0.5</max_distance>
         <fixed>ground_plane</fixed>
       </plugin>
@@ -324,3 +343,36 @@
     </gazebo>
   </xacro:if>
+  <gazebo reference="camera_link">
+    <sensor type="depth" name="depth_camera">
+      <update_rate>60</update_rate>
+      <visualize>false</visualize>
+      <camera>
+        <horizontal_fov>1.92</horizontal_fov>
+        <image>
+          <width>640</width>
+          <height>480</height>
+          <format>B8G8R8</format>
+        </image>
+        <depth_camera>
+        </depth_camera>
+        <clip>
+          <near>0.02</near>
+          <far>300</far>
+        </clip>
+        <noise>
+          <type>gaussian</type>
+          <mean>0.0</mean>
+          <stddev>0.007</stddev>
+        </noise>
+      </camera>
+      <plugin name="camera_controller" filename="libgazebo_ros_camera.so">
+        <ros>
+          <namespace>/</namespace>
+        </ros>
+        <camera_name>depth_camera</camera_name>
+        <min_depth>0.1</min_depth>
+        <max_depth>500</max_depth>
+      </plugin>
+    </sensor>
+  </gazebo>
 </robot>
